File: PCB/Alarm Clock V1.kicad_pcb (KiCad board)
At the start: 2 copper layers, 69.1 x 73.9 mm, 88 parts, among them P1 CONN_01X02, P2 CONN_01X05, P3 CONN_01X08, P6 CONN_01X02, Q1 IRLIB9343, Q10 2N3904, Q11 2N3906, Q12 2N3906, Q13 2N3904, Q14 2N3904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

Commit message: Updated PCB - Final version that was sent to fab
Parts:
- moved R7 2.81 mm to (100.1, 86.6)
- moved R8 1.80 mm to (100.1, 89.4)
- moved R9 1.05 mm to (100.1, 92.2)
- moved R10 0.57 mm to (100.1, 95.0)
- moved W5 0.25 mm to (98.3, 71.6)
- renumbered DH3 to REF**, DH6 to REF**, DH1 to REF**, DH4 to REF**, DH5 to REF**, DH2 to REF**
Routing:
- net /LEDSelect/a: track 5.82 -> 4.41 mm
- net /LEDSelect/P5: track 38.5 -> 37.1 mm
- net /LEDSelect/P13: track 9.03 -> 7.79 mm
- net /LEDSelect/b: track 5.30 -> 4.31 mm
- net /LEDSelect/c: track 4.88 -> 4.20 mm
- net Net-(Q4-Pad2): track 4.05 -> 4.62 mm
Other:
- board text added: ":µ"
- board text removed: "µ"
